File: ccd_pcb/ccd_pcb.sch (KiCad schematic (older format))
At the start: 19 parts

Commit message: do more scematics work
Parts:
- added C? (x10): 1µF, symbol C
- added C? (x7): .1µF, symbol C
- added R? (x2): 1.5k, symbol R
- added S?: ar0330CM, symbol ar0330CM
- added U? (x2): Z-TURN-LITE, symbol Z-TURN-LITE
- added U?: ADP150-2.8, symbol ADP150-2.8
Connections:
- net labels added: 1V8, 5V
- net labels removed: +1V8, +5V
- wire segments 47 -> 278
Other:
- note added: "CCD\n"
- note added: "Power\n"
- note added: "Z-Turn-Lite\n"
- note removed: "CCD Power\n"
- moved on the sheet: C?, R?, S?, U?

Commit message: route power for plugin connector
Parts:
- added C?: PCIe-36-Axiom, symbol PCIe-36-Axiom
Connections:
- wire segments 278 -> 158

Commit message: add LVDS connections to plugin connector
Connections:
- net labels added: P_N_LN0, P_N_LN1, P_N_LN2, P_N_LN3, P_N_LN4, P_N_LN5, P_N_LP0, P_N_LP1, P_N_LP2, P_N_LP3, P_N_LP4, P_N_LP5
- wire segments 158 -> 244
Other:
- note added: "Plugin Connector North"

Commit message: add connections for the extention modules
Parts:
- removed C?: PCIe-36-Axiom, symbol PCIe-36-Axiom
- added C?: Extension South, symbol PCIe-36-Axiom
- added C?: Extension North, symbol PCIe-36-Axiom
Connections:
- net labels added: EXT_VCC, IO0_N, IO0_S, IO1_N, IO1_S, IO2_N, IO2_S, IO3_N, IO3_S, IO4_N, IO4_S, IO5_N, IO5_S, IO6_N, IO6_S, IO7_N, IO7_S, IOVCC, LVDS_0A_N, LVDS_0A_S, LVDS_0B_N, LVDS_0B_S, LVDS_1A_N, LVDS_1A_S, LVDS_1B_N, LVDS_1B_S, LVDS_2A_N, LVDS_2A_S, LVDS_2B_N, LVDS_2B_S, LVDS_3A_N, LVDS_3A_S, LVDS_3B_N, LVDS_3B_S, LVDS_4A_N, LVDS_4A_S, LVDS_4B_N, LVDS_4B_S, LVDS_5A_N, LVDS_5A_S, LVDS_5B_N, LVDS_5B_S, SCL, SDA, V_I2C_N, V_I2C_S
- net labels removed: P_N_LN0, P_N_LN1, P_N_LN2, P_N_LN3, P_N_LN4, P_N_LN5, P_N_LP0, P_N_LP1, P_N_LP2, P_N_LP3, P_N_LP4, P_N_LP5
- wire segments 244 -> 242
Other:
- note added: "TODO: generate 3v3"
- note removed: "Plugin Connector North"
