File: ccd_pcb/ccd_pcb.sch (KiCad schematic (older format))
At the start: 33 parts, among them U1 Z-TURN-LITE, U2 ADP150-2.8, U3 TXS0108E, U4 TXS0108E, U5 TXS0108E

Commit message: correct the reference designators
Parts:
- renumbered U1 to A1, C12 to C10, C13 to C11, C14 to C12, C15 to C13, C16 to C14, C17 to C15, C18 to C16, C10 to C8, C11 to C9, C8 to J1, C9 to J2, PMOD1 to J3, PMOD2 to J4, PMOD3 to J5, R2 to R1, R4 to R2, R5 to R3, R6 to R4, S1 to U1
Changed lines of the file:
@@
 $EndDescr
-$Comp
-L ar0330CM S1
-U 1 1 5A471BC0
-P 2950 2700
-F 0 "S1" H 2950 2750 60  0000 C CNN
-F 1 "ar0330CM" H 2900 2900 60  0000 C CNN
-F 2 "" H 2800 4550 60  0001 C CNN
-F 3 "" H 2800 4550 60  0001 C CNN
-	1    2950 2700
-	1    0    0    -1
-$EndComp
 $Comp
 L C C1
@@
 $EndComp
 $Comp
-L C C10
+L C C8
 U 1 1 5A4745A6
 P 7350 2350
-F 0 "C10" H 7375 2450 50  0000 L CNN
+F 0 "C8" H 7375 2450 50  0000 L CNN
 F 1 "1µF" H 7375 2250 50  0000 L CNN
 F 2 "" H 7388 2200 50  0001 C CNN
@@
 $EndComp
 $Comp
-L C C11
+L C C9
 U 1 1 5A4745B2
 P 7550 2350
-F 0 "C11" H 7575 2450 50  0000 L CNN
+F 0 "C9" H 7575 2450 50  0000 L CNN
 F 1 ".1µF" H 7575 2250 50  0000 L CNN
 F 2 "" H 7588 2200 50  0001 C CNN
@@
 VDD_IO
 $Comp
-L C C12
+L C C10
 U 1 1 5A474623
 P 7900 2350
-F 0 "C12" H 7925 2450 50  0000 L CNN
+F 0 "C10" H 7925 2450 50  0000 L CNN
 F 1 "1µF" H 7925 2250 50  0000 L CNN
 F 2 "" H 7938 2200 50  0001 C CNN
@@
 $EndComp
 $Comp
-L C C14
+L C C12
 U 1 1 5A47462F
 P 8100 2350
-F 0 "C14" H 8125 2450 50  0000 L CNN
+F 0 "C12" H 8125 2450 50  0000 L CNN
 F 1 ".1µF" H 8125 2250 50  0000 L CNN
 F 2 "" H 8138 2200 50  0001 C CNN
@@
 $EndComp
 $Comp
-L C C15
+L C C13
 U 1 1 5A474685
 P 8450 2350
-F 0 "C15" H 8475 2450 50  0000 L CNN
+F 0 "C13" H 8475 2450 50  0000 L CNN
 F 1 "1µF" H 8475 2250 50  0000 L CNN
 F 2 "" H 8488 2200 50  0001 C CNN
@@
 $EndComp
 $Comp
-L C C16
+L C C14
 U 1 1 5A474691
 P 8650 2350
-F 0 "C16" H 8675 2450 50  0000 L CNN
+F 0 "C14" H 8675 2450 50  0000 L CNN
 F 1 ".1µF" H 8675 2250 50  0000 L CNN
 F 2 "" H 8688 2200 50  0001 C CNN
@@
 $EndComp
 $Comp
-L C C17
+L C C15
 U 1 1 5A475A62
 P 9000 2350
-F 0 "C17" H 9025 2450 50  0000 L CNN
+F 0 "C15" H 9025 2450 50  0000 L CNN
 F 1 "1µF" H 9025 2250 50  0000 L CNN
 F 2 "" H 9038 2200 50  0001 C CNN
@@
 $EndComp
 $Comp
-L C C18
+L C C16
 U 1 1 5A475A6E
 P 9200 2350
-F 0 "C18" H 9225 2450 50  0000 L CNN
+F 0 "C16" H 9225 2450 50  0000 L CNN
 F 1 ".1µF" H 9225 2250 50  0000 L CNN
 F 2 "" H 9238 2200 50  0001 C CNN
@@
 $EndComp
 $Comp
-L C C13
+L C C11
 U 1 1 5A478450
 P 8050 950
-F 0 "C13" H 8075 1050 50  0000 L CNN
+F 0 "C11" H 8075 1050 50  0000 L CNN
 F 1 "1µF" H 8075 850 50  0000 L CNN
 F 2 "" H 8088 800 50  0001 C CNN
@@
 $EndComp
 $Comp
-L Z-TURN-LITE U1
+L Z-TURN-LITE A1
 U 1 1 5A47B65D
 P 3000 8150
-F 0 "U1" H 3100 8050 60  0000 C CNN
+F 0 "A1" H 3100 8050 60  0000 C CNN
 F 1 "Z-TURN-LITE" H 3100 8150 60  0000 C CNN
 F 2 "" H 3250 6750 60  0001 C CNN
@@
 $EndComp
 $Comp
-L R R2
+L R R1
 U 1 1 5A4A8131
 P 1650 2050
-F 0 "R2" V 1730 2050 50  0000 C CNN
+F 0 "R1" V 1730 2050 50  0000 C CNN
 F 1 "1.5k" V 1650 2050 50  0000 C CNN
 F 2 "" V 1580 2050 50  0001 C CNN
@@
 $EndComp
 $Comp
-L R R4
+L R R2
 U 1 1 5A4A8132
 P 1850 2050
-F 0 "R4" V 1930 2050 50  0000 C CNN
+F 0 "R2" V 1930 2050 50  0000 C CNN
 F 1 "1.5k " V 1850 2050 50  0000 C CNN
 F 2 "" V 1780 2050 50  0001 C CNN
@@
 $EndComp
 $Comp
-L GNDA #PWR04
+L GNDA #PWR03
 U 1 1 5A4A8135
 P 1350 4150
-F 0 "#PWR04" H 1350 3900 50  0001 C CNN
+F 0 "#PWR03" H 1350 3900 50  0001 C CNN
 F 1 "GNDA" H 1350 4000 50  0000 C CNN
 F 2 "" H 1350 4150 50  0001 C CNN
@@
 $EndComp
 $Comp
-L GNDA #PWR05
+L GNDA #PWR04
 U 1 1 5A4A8137
 P 5600 2500
-F 0 "#PWR05" H 5600 2250 50  0001 C CNN
+F 0 "#PWR04" H 5600 2250 50  0001 C CNN
 F 1 "GNDA" H 5600 2350 50  0000 C CNN
 F 2 "" H 5600 2500 50  0001 C CNN
@@
 VDD
 $Comp
-L GNDA #PWR06
+L GNDA #PWR05
 U 1 1 5A4A813A
 P 6150 2500
-F 0 "#PWR06" H 6150 2250 50  0001 C CNN
+F 0 "#PWR05" H 6150 2250 50  0001 C CNN
 F 1 "GNDA" H 6150 2350 50  0000 C CNN
 F 2 "" H 6150 2500 50  0001 C CNN
@@
 VAA_PIX
 $Comp
-L GNDD #PWR07
+L GNDD #PWR06
 U 1 1 5A4A813D
 P 6800 2500
-F 0 "#PWR07" H 6800 2250 50  0001 C CNN
+F 0 "#PWR06" H 6800 2250 50  0001 C CNN
 F 1 "GNDD" H 6800 2350 50  0000 C CNN
 F 2 "" H 6800 2500 50  0001 C CNN
@@
 VDD
 $Comp
-L GNDD #PWR08
+L GNDD #PWR07
 U 1 1 5A4A8140
 P 7350 2500
-F 0 "#PWR08" H 7350 2250 50  0001 C CNN
+F 0 "#PWR07" H 7350 2250 50  0001 C CNN
 F 1 "GNDD" H 7350 2350 50  0000 C CNN
 F 2 "" H 7350 2500 50  0001 C CNN
@@
 $EndComp
 $Comp
-L GNDD #PWR09
+L GNDD #PWR08
 U 1 1 5A4A8143
 P 7900 2500
-F 0 "#PWR09" H 7900 2250 50  0001 C CNN
+F 0 "#PWR08" H 7900 2250 50  0001 C CNN
 F 1 "GNDD" H 7900 2350 50  0000 C CNN
 F 2 "" H 7900 2500 50  0001 C CNN
@@
 VDD_HISPI
 $Comp
-L GNDD #PWR010
+L GNDD #PWR09
 U 1 1 5A4A8146
 P 8450 2500
-F 0 "#PWR010" H 8450 2250 50  0001 C CNN
+F 0 "#PWR09" H 8450 2250 50  0001 C CNN
 F 1 "GNDD" H 8450 2350 50  0000 C CNN
 F 2 "" H 8450 2500 50  0001 C CNN
@@
 VDD_HISPI_TX
 $Comp
-L GNDD #PWR011
+L GNDD #PWR010
 U 1 1 5A4A8149
 P 9000 2500
-F 0 "#PWR011" H 9000 2250 50  0001 C CNN
+F 0 "#PWR010" H 9000 2250 50  0001 C CNN
 F 1 "GNDD" H 9000 2350 50  0000 C CNN
 F 2 "" H 9000 2500 50  0001 C CNN
@@
 VDD_PLL
 $Comp
-L GNDD #PWR012
+L GNDD #PWR011
 U 1 1 5A4A814C
 P 7300 1500
-F 0 "#PWR012" H 7300 1250 50  0001 C CNN
+F 0 "#PWR011" H 7300 1250 50  0001 C CNN
 F 1 "GNDD" H 7300 1375 50  0000 C CNN
 F 2 "" H 7300 1500 50  0001 C CNN
@@
 2V8
 $Comp
-L GNDD #PWR013
+L GNDD #PWR012
 U 1 1 5A4A814E
 P 6700 1300
-F 0 "#PWR013" H 6700 1050 50  0001 C CNN
+F 0 "#PWR012" H 6700 1050 50  0001 C CNN
 F 1 "GNDD" H 6700 1175 50  0000 C CNN
 F 2 "" H 6700 1300 50  0001 C CNN
@@
 $EndComp
 $Comp
-L GNDD #PWR014
+L GNDD #PWR013
 U 1 1 5A4A8150
 P 8050 1100
-F 0 "#PWR014" H 8050 850 50  0001 C CNN
+F 0 "#PWR013" H 8050 850 50  0001 C CNN
 F 1 "GNDD" H 8050 975 50  0000 C CNN
 F 2 "" H 8050 1100 50  0001 C CNN
@@
 Z-Turn-Lite\n
 $Comp
-L PCIe-36-Axiom C9
+L PCIe-36-Axiom J2
 U 1 1 5A47BF85
 P 7300 6800
-F 0 "C9" H 7250 6825 60  0000 C CNN
+F 0 "J2" H 7250 6825 60  0000 C CNN
 F 1 "Extension South" H 7250 6975 60  0000 C CNN
 F 2 "" H 6950 7200 60  0001 C CNN
@@
 $EndComp
 $Comp
-L GNDD #PWR016
+L GNDD #PWR014
 U 1 1 5A47BF90
 P 8750 7650
-F 0 "#PWR016" H 8750 7400 50  0001 C CNN
+F 0 "#PWR014" H 8750 7400 50  0001 C CNN
 F 1 "GNDD" H 8750 7525 50  0000 C CNN
 F 2 "" H 8750 7650 50  0001 C CNN
@@
 LVDS_0A_S
 $Comp
-L PCIe-36-Axiom C8
+L PCIe-36-Axiom J1
 U 1 1 5A484786
 P 7300 4350
-F 0 "C8" H 7250 4375 60  0000 C CNN
+F 0 "J1" H 7250 4375 60  0000 C CNN
 F 1 "Extension North" H 7250 4525 60  0000 C CNN
 F 2 "" H 6950 4750 60  0001 C CNN
@@
 IO0_N
 $Comp
-L PMOD-Host-x2-GPIO PMOD1
+L PMOD-Host-x2-GPIO J3
 U 1 1 5A4D18A6
 P 12250 1200
-F 0 "PMOD1" H 12250 1150 50  0000 C CNN
+F 0 "J3" H 12250 1150 50  0000 C CNN
 F 1 "PMODx2 North" V 12550 900 50  0001 C CNN
 F 2 "" H 12300 1500 60  0000 C CNN
@@
 $EndComp
 $Comp
-L PMOD-Host-x1-GPIO PMOD3
+L PMOD-Host-x1-GPIO J5
 U 1 1 5A53E548
 P 12250 4000
-F 0 "PMOD3" H 12200 3950 50  0000 C CNN
+F 0 "J5" H 12200 3950 50  0000 C CNN
 F 1 "PMOD-Host-x1-GPIO" V 12500 4400 50  0001 C CNN
 F 2 "" H 12300 4300 60  0000 C CNN
@@
 $EndComp
 $Comp
-L GNDA #PWR017
+L GNDA #PWR015
 U 1 1 5A5438DB
 P 5700 900
-F 0 "#PWR017" H 5700 650 50  0001 C CNN
+F 0 "#PWR015" H 5700 650 50  0001 C CNN
 F 1 "GNDA" H 5700 750 50  0000 C CNN
 F 2 "" H 5700 900 50  0001 C CNN
@@
 $EndComp
 $Comp
-L GNDD #PWR018
+L GNDD #PWR016
 U 1 1 5A543949
 P 6000 900
-F 0 "#PWR018" H 6000 650 50  0001 C CNN
+F 0 "#PWR016" H 6000 650 50  0001 C CNN
 F 1 "GNDD" H 6000 775 50  0000 C CNN
 F 2 "" H 6000 900 50  0001 C CNN
@@
 1V8
 $Comp
-L PMOD-Host-x2-GPIO PMOD2
+L PMOD-Host-x2-GPIO J4
 U 1 1 5A58CAF7
 P 12250 2600
-F 0 "PMOD2" H 12250 2550 50  0000 C CNN
+F 0 "J4" H 12250 2550 50  0000 C CNN
 F 1 "PMODx2 North" V 12550 2300 50  0001 C CNN
 F 2 "" H 12300 2900 60  0000 C CNN
@@
 PMOD7_S
 $Comp
-L GNDD #PWR019
+L GNDD #PWR017
 U 1 1 5A58FFF7
 P 12000 4550
-F 0 "#PWR019" H 12000 4300 50  0001 C CNN
+F 0 "#PWR017" H 12000 4300 50  0001 C CNN
 F 1 "GNDD" H 12000 4425 50  0000 C CNN
 F 2 "" H 12000 4550 50  0001 C CNN
@@
 $EndComp
 $Comp
-L R R6
+L R R4
 U 1 1 5A5A4F9D
 P 13150 4450
-F 0 "R6" V 13230 4450 50  0000 C CNN
+F 0 "R4" V 13230 4450 50  0000 C CNN
 F 1 "100" V 13150 4450 50  0000 C CNN
 F 2 "" V 13080 4450 50  0001 C CNN
@@
 $EndComp
 $Comp
-L R R5
+L R R3
 U 1 1 5A5A555D
 P 13150 4150
-F 0 "R5" V 13230 4150 50  0000 C CNN
+F 0 "R3" V 13230 4150 50  0000 C CNN
 F 1 "100" V 13150 4150 50  0000 C CNN
 F 2 "" V 13080 4150 50  0001 C CNN
@@
 LED1
 $Comp
-L GNDD #PWR020
+L GNDD #PWR018
 U 1 1 5A4A8154
 P 1350 10750
-F 0 "#PWR020" H 1350 10500 50  0001 C CNN
+F 0 "#PWR018" H 1350 10500 50  0001 C CNN
 F 1 "GNDD" H 1350 10625 50  0000 C CNN
 F 2 "" H 1350 10750 50  0001 C CNN
@@
 $EndComp
 $Comp
-L GNDD #PWR021
+L GNDD #PWR019
 U 1 1 5A484791
 P 8750 5200
-F 0 "#PWR021" H 8750 4950 50  0001 C CNN
+F 0 "#PWR019" H 8750 4950 50  0001 C CNN
 F 1 "GNDD" H 8750 5075 50  0000 C CNN
 F 2 "" H 8750 5200 50  0001 C CNN
@@
 	2100 2550 2100 2750
 $Comp
-L GNDD #PWR?
+L GNDD #PWR020
 U 1 1 5A5E5EB3
 P 2100 2950
-F 0 "#PWR?" H 2100 2700 50  0001 C CNN
+F 0 "#PWR020" H 2100 2700 50  0001 C CNN
 F 1 "GNDD" H 2100 2825 50  0000 C CNN
 F 2 "" H 2100 2950 50  0001 C CNN
@@
 	3950 6550 3900 6550
 Connection ~ 3950 7050
+$Comp
+L ar0330CM U1
+U 1 1 5A471BC0
+P 2950 2700
+F 0 "U1" H 2950 2750 60  0000 C CNN
+F 1 "ar0330CM" H 2900 2900 60  0000 C CNN
+F 2 "" H 2800 4550 60  0001 C CNN
+F 3 "" H 2800 4550 60  0001 C CNN
+	1    2950 2700
+	1    0    0    -1
+$EndComp
 $EndSCHEMATC

Commit message: add component footprint mappings
Parts:
- A1: footprint (none) -> parts:CONN_BTH-060-XX-X-D-LC
- C1, C10, C11, C12, C13, C14, C15, C16, C2, C3, C4, C5, C6, C7, C8, C9: footprint (none) -> Capacitors_SMD:C_0805
- D1, D2: footprint (none) -> LEDs:LED_0603_HandSoldering
- J1, J2: footprint (none) -> pcie:PCIE-36-NOPEG
- J3, J4: footprint (none) -> pmod-conn_6x2:pmod_pin_array_6x2
- J5: footprint (none) -> Pin_Headers:Pin_Header_Straight_1x06_Pitch2.54mm
- R1, R2, R3, R4: footprint (none) -> Resistors_SMD:R_0805_HandSoldering
- U2: footprint (none) -> TO_SOT_Packages_SMD:TSOT-23-5
- U3, U4, U5: footprint (none) -> Housings_SSOP:TSSOP-20_4.4x6.5mm_Pitch0.65mm
Changed lines of the file:
@@
 F 0 "C1" H 5625 2450 50  0000 L CNN
 F 1 "1µF" H 5625 2250 50  0000 L CNN
-F 2 "" H 5638 2200 50  0001 C CNN
+F 2 "Capacitors_SMD:C_0805" H 5638 2200 50  0001 C CNN
 F 3 "" H 5600 2350 50  0001 C CNN
 	1    5600 2350
@@
 F 0 "C2" H 5825 2450 50  0000 L CNN
 F 1 ".1µF" H 5825 2250 50  0000 L CNN
-F 2 "" H 5838 2200 50  0001 C CNN
+F 2 "Capacitors_SMD:C_0805" H 5838 2200 50  0001 C CNN
 F 3 "" H 5800 2350 50  0001 C CNN
 	1    5800 2350
@@
 F 0 "C3" H 6175 2450 50  0000 L CNN
 F 1 "1µF" H 6175 2250 50  0000 L CNN
-F 2 "" H 6188 2200 50  0001 C CNN
+F 2 "Capacitors_SMD:C_0805" H 6188 2200 50  0001 C CNN
 F 3 "" H 6150 2350 50  0001 C CNN
 	1    6150 2350
@@
 F 0 "C4" H 6375 2450 50  0000 L CNN
 F 1 ".1µF" H 6375 2250 50  0000 L CNN
-F 2 "" H 6388 2200 50  0001 C CNN
+F 2 "Capacitors_SMD:C_0805" H 6388 2200 50  0001 C CNN
 F 3 "" H 6350 2350 50  0001 C CNN
 	1    6350 2350
@@
 F 0 "C6" H 6825 2450 50  0000 L CNN
 F 1 "1µF" H 6825 2250 50  0000 L CNN
-F 2 "" H 6838 2200 50  0001 C CNN
+F 2 "Capacitors_SMD:C_0805" H 6838 2200 50  0001 C CNN
 F 3 "" H 6800 2350 50  0001 C CNN
 	1    6800 2350
@@
 F 0 "C7" H 7025 2450 50  0000 L CNN
 F 1 ".1µF" H 7025 2250 50  0000 L CNN
-F 2 "" H 7038 2200 50  0001 C CNN
+F 2 "Capacitors_SMD:C_0805" H 7038 2200 50  0001 C CNN
 F 3 "" H 7000 2350 50  0001 C CNN
 	1    7000 2350
@@
 F 0 "C8" H 7375 2450 50  0000 L CNN
 F 1 "1µF" H 7375 2250 50  0000 L CNN
-F 2 "" H 7388 2200 50  0001 C CNN
+F 2 "Capacitors_SMD:C_0805" H 7388 2200 50  0001 C CNN
 F 3 "" H 7350 2350 50  0001 C CNN
 	1    7350 2350
@@
 F 0 "C9" H 7575 2450 50  0000 L CNN
 F 1 ".1µF" H 7575 2250 50  0000 L CNN
-F 2 "" H 7588 2200 50  0001 C CNN
+F 2 "Capacitors_SMD:C_0805" H 7588 2200 50  0001 C CNN
 F 3 "" H 7550 2350 50  0001 C CNN
 	1    7550 2350
@@
 F 0 "C10" H 7925 2450 50  0000 L CNN
 F 1 "1µF" H 7925 2250 50  0000 L CNN
-F 2 "" H 7938 2200 50  0001 C CNN
+F 2 "Capacitors_SMD:C_0805" H 7938 2200 50  0001 C CNN
 F 3 "" H 7900 2350 50  0001 C CNN
 	1    7900 2350
@@
 F 0 "C12" H 8125 2450 50  0000 L CNN
 F 1 ".1µF" H 8125 2250 50  0000 L CNN
-F 2 "" H 8138 2200 50  0001 C CNN
+F 2 "Capacitors_SMD:C_0805" H 8138 2200 50  0001 C CNN
 F 3 "" H 8100 2350 50  0001 C CNN
 	1    8100 2350
@@
 F 0 "C13" H 8475 2450 50  0000 L CNN
 F 1 "1µF" H 8475 2250 50  0000 L CNN
-F 2 "" H 8488 2200 50  0001 C CNN
+F 2 "Capacitors_SMD:C_0805" H 8488 2200 50  0001 C CNN
 F 3 "" H 8450 2350 50  0001 C CNN
 	1    8450 2350
@@
 F 0 "C14" H 8675 2450 50  0000 L CNN
 F 1 ".1µF" H 8675 2250 50  0000 L CNN
-F 2 "" H 8688 2200 50  0001 C CNN
+F 2 "Capacitors_SMD:C_0805" H 8688 2200 50  0001 C CNN
 F 3 "" H 8650 2350 50  0001 C CNN
 	1    8650 2350
@@
 F 0 "C15" H 9025 2450 50  0000 L CNN
 F 1 "1µF" H 9025 2250 50  0000 L CNN
-F 2 "" H 9038 2200 50  0001 C CNN
+F 2 "Capacitors_SMD:C_0805" H 9038 2200 50  0001 C CNN
 F 3 "" H 9000 2350 50  0001 C CNN
 	1    9000 2350
@@
 F 0 "C16" H 9225 2450 50  0000 L CNN
 F 1 ".1µF" H 9225 2250 50  0000 L CNN
-F 2 "" H 9238 2200 50  0001 C CNN
+F 2 "Capacitors_SMD:C_0805" H 9238 2200 50  0001 C CNN
 F 3 "" H 9200 2350 50  0001 C CNN
 	1    9200 2350
@@
 F 0 "U2" H 7550 750 59  0000 C CNN
 F 1 "ADP150-2.8" H 7300 1350 59  0000 C CNN
-F 2 "" H 7200 1000 39  0000 C CNN
+F 2 "TO_SOT_Packages_SMD:TSOT-23-5" H 7200 1000 39  0001 C CNN
 F 3 "" H 7200 1000 39  0000 C CNN
 	1    7300 1000
@@
 F 0 "C11" H 8075 1050 50  0000 L CNN
 F 1 "1µF" H 8075 850 50  0000 L CNN
-F 2 "" H 8088 800 50  0001 C CNN
+F 2 "Capacitors_SMD:C_0805" H 8088 800 50  0001 C CNN
 F 3 "" H 8050 950 50  0001 C CNN
 	1    8050 950
@@
 F 0 "A1" H 3100 8050 60  0000 C CNN
 F 1 "Z-TURN-LITE" H 3100 8150 60  0000 C CNN
-F 2 "" H 3250 6750 60  0001 C CNN
+F 2 "parts:CONN_BTH-060-XX-X-D-LC" H 3250 6750 60  0001 C CNN
 F 3 "" H 3250 6750 60  0001 C CNN
 	1    3000 8150
@@
 F 0 "R1" V 1730 2050 50  0000 C CNN
 F 1 "1.5k" V 1650 2050 50  0000 C CNN
-F 2 "" V 1580 2050 50  0001 C CNN
+F 2 "Resistors_SMD:R_0805_HandSoldering" V 1580 2050 50  0001 C CNN
 F 3 "" H 1650 2050 50  0001 C CNN
 	1    1650 2050
@@
 F 0 "R2" V 1930 2050 50  0000 C CNN
 F 1 "1.5k " V 1850 2050 50  0000 C CNN
-F 2 "" V 1780 2050 50  0001 C CNN
+F 2 "Resistors_SMD:R_0805_HandSoldering" V 1780 2050 50  0001 C CNN
 F 3 "" H 1850 2050 50  0001 C CNN
 	1    1850 2050
@@
 F 0 "J2" H 7250 6825 60  0000 C CNN
 F 1 "Extension South" H 7250 6975 60  0000 C CNN
-F 2 "" H 6950 7200 60  0001 C CNN
+F 2 "pcie:PCIE-36-NOPEG" H 6950 7200 60  0001 C CNN
 F 3 "" H 6950 7200 60  0001 C CNN
 	1    7300 6800
@@
 F 0 "J1" H 7250 4375 60  0000 C CNN
 F 1 "Extension North" H 7250 4525 60  0000 C CNN
-F 2 "" H 6950 4750 60  0001 C CNN
+F 2 "pcie:PCIE-36-NOPEG" H 6950 4750 60  0001 C CNN
 F 3 "" H 6950 4750 60  0001 C CNN
 	1    7300 4350
@@
 F 0 "J3" H 12250 1150 50  0000 C CNN
 F 1 "PMODx2 North" V 12550 900 50  0001 C CNN
-F 2 "" H 12300 1500 60  0000 C CNN
+F 2 "pmod-conn_6x2:pmod_pin_array_6x2" H 12300 1500 60  0001 C CNN
 F 3 "" H 12300 1500 60  0000 C CNN
 	1    12250 1200
@@
 F 0 "D1" H 13450 4250 50  0000 C CNN
 F 1 "LED" H 13450 4050 50  0000 C CNN
-F 2 "" H 13450 4150 50  0001 C CNN
+F 2 "LEDs:LED_0603_HandSoldering" H 13450 4150 50  0001 C CNN
 F 3 "" H 13450 4150 50  0001 C CNN
 	1    13450 4150
@@
 F 0 "C5" H 6725 1250 50  0000 L CNN
 F 1 "1µF" H 6725 1050 50  0000 L CNN
-F 2 "" H 6738 1000 50  0001 C CNN
+F 2 "Capacitors_SMD:C_0805" H 6738 1000 50  0001 C CNN
 F 3 "" H 6700 1150 50  0001 C CNN
 	1    6700 1150
@@
 F 0 "J5" H 12200 3950 50  0000 C CNN
 F 1 "PMOD-Host-x1-GPIO" V 12500 4400 50  0001 C CNN
-F 2 "" H 12300 4300 60  0000 C CNN
+F 2 "Pin_Headers:Pin_Header_Straight_1x06_Pitch2.54mm" H 12300 4300 60  0001 C CNN
 F 3 "" H 12300 4300 60  0000 C CNN
 	1    12250 4000
@@
 F 0 "U3" H 10950 600 60  0000 C CNN
 F 1 "TXS0108E" H 10950 1800 60  0000 C CNN
-F 2 "" H 10950 1250 60  0001 C CNN
+F 2 "Housings_SSOP:TSSOP-20_4.4x6.5mm_Pitch0.65mm" H 10950 1250 60  0001 C CNN
 F 3 "" H 10950 1250 60  0001 C CNN
 	1    10950 1250
@@
 F 0 "J4" H 12250 2550 50  0000 C CNN
 F 1 "PMODx2 North" V 12550 2300 50  0001 C CNN
-F 2 "" H 12300 2900 60  0000 C CNN
+F 2 "pmod-conn_6x2:pmod_pin_array_6x2" H 12300 2900 60  0001 C CNN
 F 3 "" H 12300 2900 60  0000 C CNN
 	1    12250 2600
@@
 F 0 "U5" H 10950 3400 60  0000 C CNN
 F 1 "TXS0108E" H 10950 4600 60  0000 C CNN
-F 2 "" H 10950 4050 60  0001 C CNN
+F 2 "Housings_SSOP:TSSOP-20_4.4x6.5mm_Pitch0.65mm" H 10950 4050 60  0001 C CNN
 F 3 "" H 10950 4050 60  0001 C CNN
 	1    10950 4050
@@
 F 0 "U4" H 10950 2000 60  0000 C CNN
 F 1 "TXS0108E" H 10950 3200 60  0000 C CNN
-F 2 "" H 10950 2650 60  0001 C CNN
+F 2 "Housings_SSOP:TSSOP-20_4.4x6.5mm_Pitch0.65mm" H 10950 2650 60  0001 C CNN
 F 3 "" H 10950 2650 60  0001 C CNN
 	1    10950 2650
@@
 F 0 "D2" H 13450 4550 50  0000 C CNN
 F 1 "LED" H 13450 4350 50  0000 C CNN
-F 2 "" H 13450 4450 50  0001 C CNN
+F 2 "LEDs:LED_0603_HandSoldering" H 13450 4450 50  0001 C CNN
 F 3 "" H 13450 4450 50  0001 C CNN
 	1    13450 4450
@@
 F 0 "R4" V 13230 4450 50  0000 C CNN
 F 1 "100" V 13150 4450 50  0000 C CNN
-F 2 "" V 13080 4450 50  0001 C CNN
+F 2 "Resistors_SMD:R_0805_HandSoldering" V 13080 4450 50  0001 C CNN
 F 3 "" H 13150 4450 50  0001 C CNN
 	1    13150 4450
@@
 F 0 "R3" V 13230 4150 50  0000 C CNN
 F 1 "100" V 13150 4150 50  0000 C CNN
-F 2 "" V 13080 4150 50  0001 C CNN
+F 2 "Resistors_SMD:R_0805_HandSoldering" V 13080 4150 50  0001 C CNN
 F 3 "" H 13150 4150 50  0001 C CNN
 	1    13150 4150

Commit message: add lvds terminating resistor (refer to #14)
Parts:
- added R? (x5): 100, symbol R
Connections:
- wire segments 254 -> 340
Other:
- moved on the sheet: C1, C10, C11, C12, C13, C14, C15, C16, C2, C3, C4, C5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

Commit message: add more capacitors. closes #20
Parts:
- added 1µ1, 1µ10, 1µ2, 1µ3, 1µ4, 1µ5, 1µ6, 1µ7, 1µ8, 1µ9: C, symbol C
- added C12, C8, C9: .1µF, Capacitors_SMD:C_0805, symbol C
- gave numbers to parts that had none: 5
- renumbered C8 to C10, C9 to C11, C10 to C13, C11 to C14, C12 to C15, C13 to C16, C14 to C17, C15 to C18, C16 to C19, C6 to C5, C5 to C6, R3 to R8, R4 to R9
Connections:
- wire segments 340 -> 283
Other:
- moved on the sheet: C5, C7

Commit message: begin layouting and routhing the board
Parts:
- C1, C10, C11, C12, C13, C14, C15, C16, C17, C18, C19, C2, C3, C4, C5, C6, C7, C8, C9: footprint Capacitors_SMD:C_0805 -> Capacitors_SMD:C_0805_HandSoldering
- C20: renamed from 1µ1; value C -> 1µ; footprint (none) -> Capacitors_SMD:C_0805_HandSoldering
- C21: renamed from 1µ2; value C -> 1µ; footprint (none) -> Capacitors_SMD:C_0805_HandSoldering
- C22: renamed from 1µ3; value C -> 1µ; footprint (none) -> Capacitors_SMD:C_0805_HandSoldering
- C23: renamed from 1µ4; value C -> 1µ; footprint (none) -> Capacitors_SMD:C_0805_HandSoldering
- C24: renamed from 1µ5; value C -> 1µ; footprint (none) -> Capacitors_SMD:C_0805_HandSoldering
- C25: renamed from 1µ6; value C -> 1µ; footprint (none) -> Capacitors_SMD:C_0805_HandSoldering
- C26: renamed from 1µ7; value C -> 1µ; footprint (none) -> Capacitors_SMD:C_0805_HandSoldering
- C27: renamed from 1µ8; value C -> 1µ; footprint (none) -> Capacitors_SMD:C_0805_HandSoldering
- C28: renamed from 1µ9; value C -> 1µ; footprint (none) -> Capacitors_SMD:C_0805_HandSoldering
- C29: renamed from 1µ10; value C -> 1µ; footprint (none) -> Capacitors_SMD:C_0805_HandSoldering
- R3, R4, R5, R6, R7: footprint (none) -> Resistors_SMD:R_0805_HandSoldering
- U1: footprint (none) -> parts:CLCC48_0.8mm
Connections:
- net labels added: LVDSn0_N, LVDSn0_P, LVDSn1_N, LVDSn1_P, LVDSn2_N, LVDSn2_P, LVDSn3_N, LVDSn3_P, LVDSn4_N, LVDSn4_P, LVDSn5_N, LVDSn5_P, LVDSs0_N, LVDSs0_P, LVDSs1_N, LVDSs1_P, LVDSs2_N, LVDSs2_P, LVDSs3_N, LVDSs3_P, LVDSs4_N, LVDSs4_P, LVDSs5_N, LVDSs5_P, SLVC_N, SLVC_P, SLVS0_N, SLVS0_P, SLVS1_N, SLVS1_P, SLVS2_N, SLVS2_P, SLVS3_N, SLVS3_P
- net labels removed: LVDS_0A_N, LVDS_0A_S, LVDS_0B_N, LVDS_0B_S, LVDS_1A_N, LVDS_1A_S, LVDS_1B_N, LVDS_1B_S, LVDS_2A_N, LVDS_2A_S, LVDS_2B_N, LVDS_2B_S, LVDS_3A_N, LVDS_3A_S, LVDS_3B_N, LVDS_3B_S, LVDS_4A_N, LVDS_4A_S, LVDS_4B_N, LVDS_4B_S, LVDS_5A_N, LVDS_5A_S, LVDS_5B_N, LVDS_5B_S

Commit message: redo layout
Parts:
- R1, R2, R3, R4, R5, R6, R7, R8, R9: footprint Resistors_SMD:R_0805_HandSoldering -> Resistors_SMD:R_0603_HandSoldering
Connections:
- net labels added: FLASH, SHUTTER, SLVSC_N, SLVSC_P
- net labels removed: SLVC_N, SLVC_P
- wire segments 283 -> 255
Other:
- moved on the sheet: R3, R4, R5, R6, R7

Commit message: most of the routing done
Parts:
- removed C8: .1µF, Capacitors_SMD:C_0805_HandSoldering, symbol C
Connections:
- wire segments 255 -> 354
Other:
- moved on the sheet: C9

Commit message: closes #21;
Connections:
- wire segments 354 -> 255
