File: ccd_pcb/ccd_pcb.sch (KiCad schematic (older format))
At the start: 50 parts, among them J1 Extension North, J2 Extension South, J3 PMODx2 North, J4 PMODx2 North, J5 PMOD-Host-x1-GPIO, U1 ar0330CM, U2 ADP150-2.8, U3 TXS0108E, U4 TXS0108E, U5 TXS0108E

Commit message: begin working on schematic v2
Parts:
- removed A1: Z-TURN-LITE, parts:CONN_BTH-060-XX-X-D-LC, symbol Z-TURN-LITE
- removed C10, C5: 1µF, Capacitors_SMD:C_0805_HandSoldering, symbol C
- removed R3, R4, R5, R6, R7: 100, Resistors_SMD:R_0603_HandSoldering, symbol R
- added A?: Z-TURN-LITE, symbol Z-TURN-LITE
- added C? (x4): 1µF, Capacitors_SMD:C_0805_HandSoldering, symbol C
- added C? (x2): 1µ, symbol C
- added U? (x2): ADP150-2.8, TO_SOT_Packages_SMD:TSOT-23-5, symbol ADP150-2.8
- renumbered C1 to C?, C2 to C?, C3 to C?, C4 to C?, C7 to C?, C11 to C?, C13 to C?, C15 to C?, C16 to C?, C17 to C?, C18 to C?, C19 to C?, C6 to C?, C14 to C?, C12 to C?, C9 to C?, C20 to C?, C22 to C?, C21 to C?, C23 to C?, C26 to C?, C25 to C?, C24 to C?, C27 to C?, C28 to C?, C29 to C?, D1 to D?, D2 to D?, J2 to J?, J1 to J?, J3 to J?, J5 to J?, J4 to J?, R1 to R?, R2 to R?, R9 to R?, R8 to R?, U1 to U?, U2 to U?, U3 to U?, U4 to U?, U5 to U?
Connections:
- net labels added: ADDR_SELECT, CCD_CLK, CCD_TRIGGER, RESET, S_CLK, S_DATA, VDD_B34, VDD_B35
- wire segments 255 -> 338
Other:
- note removed: "Z-Turn-Lite\n"
- moved on the sheet: C?, R?, U?

Commit message: update
Parts:
- removed C? (x4): 1µF, Capacitors_SMD:C_0805_HandSoldering, symbol C
- removed C? (x7): 1µ, Capacitors_SMD:C_0805_HandSoldering, symbol C
- removed C?: 1µ, symbol C
- removed D? (x2): LED, LEDs:LED_0603_HandSoldering, symbol LED
- removed J?: PMOD-Host-x1-GPIO, Pin_Headers:Pin_Header_Straight_1x06_Pitch2.54mm, symbol PMOD-Host-x1-GPIO
- removed J?: PMODx2 North, pmod-conn_6x2:pmod_pin_array_6x2, symbol PMOD-Host-x2-GPIO
- removed R? (x2): 100, Resistors_SMD:R_0603_HandSoldering, symbol R
- removed U? (x2): ADP150-2.8, TO_SOT_Packages_SMD:TSOT-23-5, symbol ADP150-2.8
- removed U? (x2): TXS0108E, Housings_SSOP:TSSOP-20_4.4x6.5mm_Pitch0.65mm, symbol TXS0108E
- added C? (x5): 1µ, Capacitors_SMD:C_0805_HandSoldering, symbol C
- added C? (x2): 4.7µF, Capacitors_SMD:C_0805_HandSoldering, symbol C
- added C? (x2): 1µF, Capacitors_SMD:C_0805_HandSoldering, symbol C
- added C? (x2): .1µ, symbol C
- added C?: 1µ, symbol C
- added C? (x4): .1µ, Capacitors_SMD:C_0805_HandSoldering, symbol C
- added D?: ws2812, symbol ws2812
- added J?: PMODx2 North, pmod-conn_6x2:pmod_pin_array_6x2, symbol PMOD-Host-x2-GPIO
- added J?: PMOD-Host-x1-GPIO, Pin_Headers:Pin_Header_Straight_1x06_Pitch2.54mm, symbol PMOD-Host-x1-GPIO
- added R? (x2): 1.5k, Resistors_SMD:R_0603_HandSoldering, symbol R
- added U?: MCP1727-1V8, symbol MCP1727-1V8
- added U?: MCP1727-3V3, symbol MCP1727-3V3
- added U?: BMX055, symbol BMX055
- added U? (x2): TXS0108E, Housings_SSOP:TSSOP-20_4.4x6.5mm_Pitch0.65mm, symbol TXS0108E
- C?: value .1µF -> 1µF
- C? (x2): value 1µ -> .1µ
- R? (x2): value 1.5k -> 15k
Connections:
- net labels added: VDDIO_34, VDDIO_35
- net labels removed: VDD_B34, VDD_B35
- wire segments 338 -> 311
- no-connect marks 36 -> 35
Other:
- moved on the sheet: C?, R?, U?

Commit message: v2 r1
Parts:
- removed C? (x2): 1µ, symbol C
- removed C? (x2): .1µ, symbol C
- added C1, C16, C19, C2, C3, C7, C9: .1µ, symbol C
- added D2, D3, D4, D5: ws2812, symbol ws2812
- added J1, J2, J3, J7: GS3, Connectors:GS3, symbol GS3
- added R1, R2: 15k, Resistors_SMD:R_0603_HandSoldering, symbol R
- added U1: 74LVC1T45GW, symbol 74LVC1T45GW
- gave numbers to parts that had none: 51
Connections:
- net labels added: A_ADDR, A_M_ADDR, G_ADDR, IMU_SCLK, IMU_SDATA, WS2812
- net labels removed: ADDR_SELECT, FLASH, LED1, LED2
- no-connect marks 35 -> 55
Other:
- note added: "IMU"
- moved on the sheet: C10, C11, C12, C13, C14, C15, C17, C18, C20, C21, C22, C23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

Commit message: add incremental encoder and soldering training
Parts:
- added C8, C9: .01µ, Capacitors_SMD:C_0805_HandSoldering, symbol C
- added E1: EN12-VS, symbol EN12-VS
- added R3, R4, R5: 10k, Resistors_SMD:R_0603_HandSoldering, symbol R
- added R? (x100): DNP, Resistors_SMD:R_0603_HandSoldering, symbol R
- added TP1, TP2, TP3, TP4: TEST, symbol TEST
- R1, R2: value 15k -> 10k
- renumbered C8 to C10, C9 to C11, C10 to C12, C11 to C16, C12 to C17, C16 to C18, C17 to C19, C18 to C20, C19 to C21, C20 to C22, C21 to C23, C22 to C24, C23 to C25, C24 to C26, C25 to C27, C26 to C28, C27 to C29, C28 to C30, C29 to C31, C30 to C32, C31 to C33, C32 to C34, C33 to C35, C34 to C36, C35 to C37, C36 to C38, C37 to C39, C38 to C40, C39 to C41, R3 to R6, R4 to R7, R5 to R8, R6 to R9
Connections:
- net labels added: EN_A, EN_B, EN_S
- net labels removed: IMU_SCLK, IMU_SDATA
- wire segments 311 -> 322
- no-connect marks 55 -> 254
Other:
- note added: "Incremental Encoder"
- note added: "Solder training area :)"
- note added: "testpoints"
- moved on the sheet: C1, C11, C13, C14, C15, C18, C2, C21, C3, C4, C5, C6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

Commit message: small fix
Parts:
- gave numbers to parts that had none: 100
- renumbered R8 to R108, R9 to R109, R6 to R56, R7 to R57
Connections:
- wire segments 322 -> 443
- no-connect marks 254 -> 255

Commit message: more stuff
Parts:
- added C42, C43, C46: 1µF, Capacitors_SMD:C_0402, symbol C
- added C44, C45, C47: .1µF, Capacitors_SMD:C_0402, symbol C
- A1: footprint (none) -> parts:CONN_BTH-060-XX-X-D-LC
- C1, C11, C18, C2, C21, C3, C7: footprint (none) -> Capacitors_SMD:C_0402
- C10, C12, C13, C14, C15, C19, C20, C22, C23, C24, C25, C26, C27, C28, C29, C30, C31, C32, C34, C35, C36, C37, C38, C39, C4, C40, C41, C5, C6, C8, C9: footprint Capacitors_SMD:C_0805_HandSoldering -> Capacitors_SMD:C_0402
- C16, C17: footprint Capacitors_SMD:C_0805_HandSoldering -> Capacitors_SMD:C_0603_HandSoldering
- C33: value .1µF -> 1µF; footprint Capacitors_SMD:C_0805_HandSoldering -> Capacitors_SMD:C_0402
- D1, D2, D3, D4, D5: footprint (none) -> LEDs:LED_WS2812-PLCC6
- E1: footprint (none) -> parts:EN12-VS
- R10, R11, R12, R13, R14, R15, R16, R17, R18, R19, R20, R21, R22, R23, R24, R25, R26, R27, R28, R29, R30, R31, R32, R33, R34, R35, R36, R37, R38, R39, R40, R41, R42, R43, R44, R45, R46, R47, R48, R49, R50, R51, R52, R53, R54, R55, R6, R7, R8, R9: footprint Resistors_SMD:R_0603_HandSoldering -> Resistors_SMD:R_0402_NoSilk
- R100, R101, R102, R103, R104, R105, R106, R107, R58, R59, R60, R61, R62, R63, R64, R65, R66, R67, R68, R69, R70, R71, R72, R73, R74, R75, R76, R77, R78, R79, R80, R81, R82, R83, R84, R85, R86, R87, R88, R89, R90, R91, R92, R93, R94, R95, R96, R97, R98, R99: footprint Resistors_SMD:R_0603_HandSoldering -> Capacitors_SMD:C_0402_NoSilk
- TP1, TP2, TP3, TP4: footprint (none) -> Connectors_TestPoints:Test_Point_Pad_2.0x2.0mm
- U1: footprint (none) -> parts:SC-88
- U2: footprint (none) -> NQBit:BMX055
- U7, U8: footprint (none) -> Housings_SOIC:SOIC-8_3.9x4.9mm_Pitch1.27mm
Connections:
- wire segments 443 -> 333
Other:
- moved on the sheet: C23, C24, C27, C28, C32, C33, C37, C38

Commit message: update
Parts:
- removed C35, C36, C40, C41: 1µ, Capacitors_SMD:C_0402, symbol C
- added R110, R111, R112, R113: 15k, Resistors_SMD:R_0603_HandSoldering, symbol R
- C30, C31: value 1µ -> .1µF
Connections:
- wire segments 333 -> 338
Other:
- moved on the sheet: C11, C18, C21, C3, C7
