File: ccd_pcb/ccd_pcb.kicad_pcb (KiCad board)
At the start: 2 copper layers, 91 x 85 mm, 53 parts, among them J1 Extension North, J2 Extension South, J3 PMODx2 North, J5 PMOD-Host-x1-GPIO, U1 ar0330CM, U2 ADP150-2.8, U3 TXS0108E, U4 TXS0108E, U5 TXS0108E

Commit message: more stuff
Parts:
- removed ? (x4): mounting_hole, mounting_hole:mounting_hole
- removed J5: PMOD-Host-x1-GPIO, Pin_Headers:Pin_Header_Straight_1x06_Pitch2.54mm
- added C30: 1µ, Capacitors_SMD:C_0402, F.Cu at (77.9, 49.2)
- added C31: 1µ, Capacitors_SMD:C_0402, F.Cu at (86.1, 126.7)
- added C32: 1µF, Capacitors_SMD:C_0402, F.Cu at (185.9, 42.8)
- added C33: 1µF, Capacitors_SMD:C_0402, F.Cu at (173.2, 50.5)
- added C34: 1µF, Capacitors_SMD:C_0402, F.Cu at (212.5, 55.5)
- added C35: 1µ, Capacitors_SMD:C_0402, F.Cu at (88.8, 49.2)
- added C36: 1µ, Capacitors_SMD:C_0402, F.Cu at (91.2, 126.7)
- added C37: .1µF, Capacitors_SMD:C_0402, F.Cu at (189.7, 42.8)
- added C38: .1µF, Capacitors_SMD:C_0402, F.Cu at (177.0, 50.5)
- added C39: .1µF, Capacitors_SMD:C_0402, F.Cu at (215.1, 55.5)
- added C40: 1µ, Capacitors_SMD:C_0402, F.Cu at (85.0, 47.9)
- added C41: 1µ, Capacitors_SMD:C_0402, F.Cu at (97.5, 126.7)
- added C42: 1µF, Capacitors_SMD:C_0402, F.Cu at (212.5, 36.5)
- added C43: 1µF, Capacitors_SMD:C_0402, F.Cu at (173.2, 54.3)
- added C44: .1µF, Capacitors_SMD:C_0402, F.Cu at (216.3, 36.5)
- added C45: .1µF, Capacitors_SMD:C_0402, F.Cu at (177.0, 54.3)
- added C46: 1µF, Capacitors_SMD:C_0402, F.Cu at (173.2, 58.1)
- added C47: .1µF, Capacitors_SMD:C_0402, F.Cu at (177.0, 58.1)
- added C8: .01µ, Capacitors_SMD:C_0402, F.Cu at (256.4, 158.4)
- added D3: ws2812, LEDs:LED_WS2812-PLCC6, F.Cu at (272.2, 84.7)
- added D4: ws2812, LEDs:LED_WS2812-PLCC6, F.Cu at (272.2, 96.5)
- added D5: ws2812, LEDs:LED_WS2812-PLCC6, F.Cu at (271.9, 107.6)
- added E1: EN12-VS, parts:EN12-VS, F.Cu at (255.6, 149.2)
- added J4: PMODx2 North, pmod-conn_6x2:pmod_pin_array_6x2, F.Cu at (156.7, 183.8)
- added J6: PMOD-Host-x1-GPIO, Pin_Headers:Pin_Header_Straight_1x06_Pitch2.54mm, F.Cu at (91.9, 185.1)
- added J7: GS3, Connectors:GS3, F.Cu at (189.7, 13.6)
- added J8: Extension North, pcie:PCIE-36-NOPEG, F.Cu at (89.9, 35.2)
- added J9: Extension South, pcie:PCIE-36-NOPEG, F.Cu at (95.7, 117.8)
- added R10: DNP, Resistors_SMD:R_0402_NoSilk, F.Cu at (22.0, 54.3)
- added R100: DNP, Capacitors_SMD:C_0402_NoSilk, F.Cu at (22.0, 88.5)
- added R101: DNP, Capacitors_SMD:C_0402_NoSilk, F.Cu at (25.9, 88.5)
- added R102: DNP, Capacitors_SMD:C_0402_NoSilk, F.Cu at (29.7, 88.5)
- added R103: DNP, Capacitors_SMD:C_0402_NoSilk, F.Cu at (33.5, 88.5)
- added R104: DNP, Capacitors_SMD:C_0402_NoSilk, F.Cu at (37.3, 88.5)
- added R105: DNP, Capacitors_SMD:C_0402_NoSilk, F.Cu at (41.1, 88.5)
- added R106: DNP, Capacitors_SMD:C_0402_NoSilk, F.Cu at (44.9, 88.5)
- added R107: DNP, Capacitors_SMD:C_0402_NoSilk, F.Cu at (48.7, 88.5)
- added R108: 15k, Resistors_SMD:R_0603_HandSoldering, F.Cu at (137.8, 58.1)
- added R109: 15k, Resistors_SMD:R_0603_HandSoldering, F.Cu at (137.8, 54.3)
- added R11: DNP, Resistors_SMD:R_0402_NoSilk, F.Cu at (25.9, 54.3)
- added R12: DNP, Resistors_SMD:R_0402_NoSilk, F.Cu at (29.7, 54.3)
- added R13: DNP, Resistors_SMD:R_0402_NoSilk, F.Cu at (33.5, 54.3)
- added R14: DNP, Resistors_SMD:R_0402_NoSilk, F.Cu at (37.3, 54.3)
- added R15: DNP, Resistors_SMD:R_0402_NoSilk, F.Cu at (41.1, 54.3)
- added R16: DNP, Resistors_SMD:R_0402_NoSilk, F.Cu at (44.9, 54.3)
- added R17: DNP, Resistors_SMD:R_0402_NoSilk, F.Cu at (48.7, 54.3)
- added R18: DNP, Resistors_SMD:R_0402_NoSilk, F.Cu at (52.5, 54.3)
- added R19: DNP, Resistors_SMD:R_0402_NoSilk, F.Cu at (56.4, 54.3)
- added R20: DNP, Resistors_SMD:R_0402_NoSilk, F.Cu at (22.0, 58.1)
- added R21: DNP, Resistors_SMD:R_0402_NoSilk, F.Cu at (25.9, 58.1)
- added R22: DNP, Resistors_SMD:R_0402_NoSilk, F.Cu at (29.7, 58.1)
- added R23: DNP, Resistors_SMD:R_0402_NoSilk, F.Cu at (33.5, 58.1)
- added R24: DNP, Resistors_SMD:R_0402_NoSilk, F.Cu at (37.3, 58.1)
- added R25: DNP, Resistors_SMD:R_0402_NoSilk, F.Cu at (41.1, 58.1)
- added R26: DNP, Resistors_SMD:R_0402_NoSilk, F.Cu at (45.0, 58.1)
- added R27: DNP, Resistors_SMD:R_0402_NoSilk, F.Cu at (52.5, 58.1)
- added R28: DNP, Resistors_SMD:R_0402_NoSilk, F.Cu at (48.7, 58.1)
- added R29: DNP, Resistors_SMD:R_0402_NoSilk, F.Cu at (56.3, 58.1)
- added R30: DNP, Resistors_SMD:R_0402_NoSilk, F.Cu at (22.0, 61.9)
- added R31: DNP, Resistors_SMD:R_0402_NoSilk, F.Cu at (25.9, 61.9)
- added R32: DNP, Resistors_SMD:R_0402_NoSilk, F.Cu at (29.7, 61.9)
- added R33: DNP, Resistors_SMD:R_0402_NoSilk, F.Cu at (33.5, 61.9)
- added R34: DNP, Resistors_SMD:R_0402_NoSilk, F.Cu at (37.3, 61.9)
- added R35: DNP, Resistors_SMD:R_0402_NoSilk, F.Cu at (41.1, 61.9)
- added R36: DNP, Resistors_SMD:R_0402_NoSilk, F.Cu at (44.9, 61.9)
- added R37: DNP, Resistors_SMD:R_0402_NoSilk, F.Cu at (48.7, 61.9)
- added R38: DNP, Resistors_SMD:R_0402_NoSilk, F.Cu at (52.5, 61.9)
- added R39: DNP, Resistors_SMD:R_0402_NoSilk, F.Cu at (56.3, 61.9)
- added R40: DNP, Resistors_SMD:R_0402_NoSilk, F.Cu at (22.0, 65.7)
- added R41: DNP, Resistors_SMD:R_0402_NoSilk, F.Cu at (25.9, 65.7)
- added R42: DNP, Resistors_SMD:R_0402_NoSilk, F.Cu at (29.7, 65.7)
- added R43: DNP, Resistors_SMD:R_0402_NoSilk, F.Cu at (33.5, 65.7)
- added R44: DNP, Resistors_SMD:R_0402_NoSilk, F.Cu at (37.3, 65.7)
- added R45: DNP, Resistors_SMD:R_0402_NoSilk, F.Cu at (41.1, 65.7)
- added R46: DNP, Resistors_SMD:R_0402_NoSilk, F.Cu at (44.9, 65.7)
- added R47: DNP, Resistors_SMD:R_0402_NoSilk, F.Cu at (48.7, 65.7)
- added R48: DNP, Resistors_SMD:R_0402_NoSilk, F.Cu at (52.5, 65.7)
- added R49: DNP, Resistors_SMD:R_0402_NoSilk, F.Cu at (56.3, 65.7)
- added R50: DNP, Resistors_SMD:R_0402_NoSilk, F.Cu at (22.0, 69.5)
- added R51: DNP, Resistors_SMD:R_0402_NoSilk, F.Cu at (25.9, 69.5)
- added R52: DNP, Resistors_SMD:R_0402_NoSilk, F.Cu at (29.7, 69.5)
- added R53: DNP, Resistors_SMD:R_0402_NoSilk, F.Cu at (33.5, 69.5)
- added R54: DNP, Resistors_SMD:R_0402_NoSilk, F.Cu at (37.3, 69.5)
- added R55: DNP, Resistors_SMD:R_0402_NoSilk, F.Cu at (41.1, 69.5)
- added R56: 1.5k, Resistors_SMD:R_0603_HandSoldering, F.Cu at (188.2, 162.2)
- added R57: 1.5k, Resistors_SMD:R_0603_HandSoldering, F.Cu at (207.3, 162.2)
- added R58: DNP, Capacitors_SMD:C_0402_NoSilk, F.Cu at (52.5, 69.5)
- added R59: DNP, Capacitors_SMD:C_0402_NoSilk, F.Cu at (56.3, 69.5)
- added R60: DNP, Capacitors_SMD:C_0402_NoSilk, F.Cu at (22.0, 73.3)
- added R61: DNP, Capacitors_SMD:C_0402_NoSilk, F.Cu at (25.9, 73.3)
- added R62: DNP, Capacitors_SMD:C_0402_NoSilk, F.Cu at (29.7, 73.3)
- added R63: DNP, Capacitors_SMD:C_0402_NoSilk, F.Cu at (33.5, 73.3)
- added R64: DNP, Capacitors_SMD:C_0402_NoSilk, F.Cu at (37.3, 73.3)
- added R65: DNP, Capacitors_SMD:C_0402_NoSilk, F.Cu at (41.1, 73.3)
- added R66: DNP, Capacitors_SMD:C_0402_NoSilk, F.Cu at (44.9, 73.3)
- added R67: DNP, Capacitors_SMD:C_0402_NoSilk, F.Cu at (48.9, 73.3)
- added R68: DNP, Capacitors_SMD:C_0402_NoSilk, F.Cu at (52.5, 73.3)
- added R69: DNP, Capacitors_SMD:C_0402_NoSilk, F.Cu at (56.3, 73.3)
- added R70: DNP, Capacitors_SMD:C_0402_NoSilk, F.Cu at (22.0, 77.1)
- added R71: DNP, Capacitors_SMD:C_0402_NoSilk, F.Cu at (25.9, 77.1)
- added R72: DNP, Capacitors_SMD:C_0402_NoSilk, F.Cu at (29.7, 77.1)
- added R73: DNP, Capacitors_SMD:C_0402_NoSilk, F.Cu at (33.5, 77.1)
- added R74: DNP, Capacitors_SMD:C_0402_NoSilk, F.Cu at (37.3, 77.1)
- added R75: DNP, Capacitors_SMD:C_0402_NoSilk, F.Cu at (41.1, 77.1)
- added R76: DNP, Capacitors_SMD:C_0402_NoSilk, F.Cu at (44.9, 77.1)
- added R77: DNP, Capacitors_SMD:C_0402_NoSilk, F.Cu at (48.7, 77.1)
- added R78: DNP, Capacitors_SMD:C_0402_NoSilk, F.Cu at (52.5, 77.1)
- added R79: DNP, Capacitors_SMD:C_0402_NoSilk, F.Cu at (56.3, 77.1)
- added R80: DNP, Capacitors_SMD:C_0402_NoSilk, F.Cu at (22.0, 80.9)
- added R81: DNP, Capacitors_SMD:C_0402_NoSilk, F.Cu at (25.9, 80.9)
- added R82: DNP, Capacitors_SMD:C_0402_NoSilk, F.Cu at (29.7, 80.9)
- added R83: DNP, Capacitors_SMD:C_0402_NoSilk, F.Cu at (33.5, 80.9)
- added R84: DNP, Capacitors_SMD:C_0402_NoSilk, F.Cu at (37.3, 80.9)
- added R85: DNP, Capacitors_SMD:C_0402_NoSilk, F.Cu at (41.1, 80.9)
- added R86: DNP, Capacitors_SMD:C_0402_NoSilk, F.Cu at (44.9, 80.9)
- added R87: DNP, Capacitors_SMD:C_0402_NoSilk, F.Cu at (48.7, 80.9)
- added R88: DNP, Capacitors_SMD:C_0402_NoSilk, F.Cu at (52.5, 80.9)
- added R89: DNP, Capacitors_SMD:C_0402_NoSilk, F.Cu at (56.3, 80.9)
- added R90: DNP, Capacitors_SMD:C_0402_NoSilk, F.Cu at (22.0, 84.7)
- added R91: DNP, Capacitors_SMD:C_0402_NoSilk, F.Cu at (25.9, 84.7)
- added R92: DNP, Capacitors_SMD:C_0402_NoSilk, F.Cu at (29.7, 84.7)
- added R93: DNP, Capacitors_SMD:C_0402_NoSilk, F.Cu at (33.5, 84.7)
- added R94: DNP, Capacitors_SMD:C_0402_NoSilk, F.Cu at (37.3, 84.7)
- added R95: DNP, Capacitors_SMD:C_0402_NoSilk, F.Cu at (41.1, 84.7)
- added R96: DNP, Capacitors_SMD:C_0402_NoSilk, F.Cu at (44.9, 84.7)
- added R97: DNP, Capacitors_SMD:C_0402_NoSilk, F.Cu at (48.7, 84.7)
- added R98: DNP, Capacitors_SMD:C_0402_NoSilk, F.Cu at (52.5, 84.7)
- added R99: DNP, Capacitors_SMD:C_0402_NoSilk, F.Cu at (56.3, 84.7)
- added TP1: TEST, Connectors_TestPoints:Test_Point_Pad_2.0x2.0mm, F.Cu at (164.3, 100.0)
- added TP2: TEST, Connectors_TestPoints:Test_Point_Pad_2.0x2.0mm, F.Cu at (161.7, 91.1)
- added TP3: TEST, Connectors_TestPoints:Test_Point_Pad_2.0x2.0mm, F.Cu at (170.6, 97.4)
- added TP4: TEST, Connectors_TestPoints:Test_Point_Pad_2.0x2.0mm, F.Cu at (169.4, 89.8)
- added U6: ADP150-2.8, TO_SOT_Packages_SMD:TSOT-23-5, F.Cu at (224.0, 157.1)
- added U7: MCP1727-1V8, Housings_SOIC:SOIC-8_3.9x4.9mm_Pitch1.27mm, F.Cu at (184.6, 155.9)
- added U8: MCP1727-3V3, Housings_SOIC:SOIC-8_3.9x4.9mm_Pitch1.27mm, F.Cu at (204.9, 155.9)
- added U9: ar0330CM, parts:CLCC48_0.8mm, F.Cu at (190.9, 26.3)
- C1, C13, C14, C18: value 1µF -> .1µ; footprint Capacitors_SMD:C_0805_HandSoldering -> Capacitors_SMD:C_0402; moved to F.Cu
- C10: footprint Capacitors_SMD:C_0805_HandSoldering -> Capacitors_SMD:C_0402; moved to F.Cu
- C11, C15, C2, C7: value .1µF -> .1µ; footprint Capacitors_SMD:C_0805_HandSoldering -> Capacitors_SMD:C_0402; moved to F.Cu
- C12, C19: value .1µF -> 1µF; footprint Capacitors_SMD:C_0805_HandSoldering -> Capacitors_SMD:C_0402; moved to F.Cu
- C16: value 1µF -> 4.7µF; footprint Capacitors_SMD:C_0805_HandSoldering -> Capacitors_SMD:C_0603_HandSoldering
- C17: value .1µF -> 4.7µF; footprint Capacitors_SMD:C_0805_HandSoldering -> Capacitors_SMD:C_0603_HandSoldering; moved to F.Cu
- C20, C22, C24: value 1µ -> 1µF; footprint Capacitors_SMD:C_0805_HandSoldering -> Capacitors_SMD:C_0402; moved to F.Cu
- C21: value 1µ -> .1µ; footprint Capacitors_SMD:C_0805_HandSoldering -> Capacitors_SMD:C_0402; moved to F.Cu
- C23, C25: value 1µ -> 1µF; footprint Capacitors_SMD:C_0805_HandSoldering -> Capacitors_SMD:C_0402
- C26, C28, C29: value 1µ -> .1µF; footprint Capacitors_SMD:C_0805_HandSoldering -> Capacitors_SMD:C_0402
- C27: value 1µ -> .1µF; footprint Capacitors_SMD:C_0805_HandSoldering -> Capacitors_SMD:C_0402; moved to F.Cu
- C3, C5, C6: value 1µF -> .1µ; footprint Capacitors_SMD:C_0805_HandSoldering -> Capacitors_SMD:C_0402
- C4: value .1µF -> .1µ; footprint Capacitors_SMD:C_0805_HandSoldering -> Capacitors_SMD:C_0402
- C9: value .1µF -> .01µ; footprint Capacitors_SMD:C_0805_HandSoldering -> Capacitors_SMD:C_0402; moved to F.Cu
- D1, D2: value LED -> ws2812; footprint LEDs:LED_0603_HandSoldering -> LEDs:LED_WS2812-PLCC6
- J1: value Extension North -> GS3; footprint pcie:PCIE-36-NOPEG -> Connectors:GS3
- J2: value Extension South -> GS3; footprint pcie:PCIE-36-NOPEG -> Connectors:GS3
- J3: value PMODx2 North -> GS3; footprint pmod-conn_6x2:pmod_pin_array_6x2 -> Connectors:GS3
- R1, R2: value 1.5k -> 10k; moved to F.Cu
- R3, R4, R5: value 100 -> 10k
- R6, R7, R8, R9: value 100 -> DNP; footprint Resistors_SMD:R_0603_HandSoldering -> Resistors_SMD:R_0402_NoSilk
- U1: value ar0330CM -> 74LVC1T45GW; footprint parts:CLCC48_0.8mm -> parts:SC-88; moved to F.Cu
- U2: value ADP150-2.8 -> BMX055; footprint TO_SOT_Packages_SMD:TSOT-23-5 -> NQBit:BMX055
- moved D2 270.3 mm to (272.2, 74.6), turned to 270 degrees
- moved D1 270.2 mm to (272.2, 63.1), turned to 270 degrees
- moved R1 257.8 mm to (266.1, 163.5), turned to 0 degrees
- moved R2 253.6 mm to (269.9, 150.8), turned to 0 degrees
- moved C9 250.4 mm to (265.3, 158.4), turned to 0 degrees
- moved C3 248.4 mm to (270.6, 58.3), turned to 270 degrees
- moved J1 231.2 mm to (257.0, 20.0)
- moved R5 231.0 mm to (272.4, 159.7), turned to 0 degrees
- moved C7 230.7 mm to (271.2, 70.1), turned to 180 degrees
- moved U1 227.4 mm to (272.9, 48.4), turned to 270 degrees
- moved C10 226.9 mm to (221.4, 162.2), turned to 0 degrees
- moved C12 224.4 mm to (227.8, 162.2), turned to 0 degrees
- moved U2 223.4 mm to (252.4, 33.7), turned to 0 degrees
- moved C2 222.3 mm to (258.3, 32.7), turned to 0 degrees
- moved C11 221.7 mm to (265.3, 86.0), turned to 0 degrees
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Connections:
- A1 pad 1: (no net) -> Net-(A1-Pad1)
- A1 pad 103: LED2 -> CCD_CLK
- A1 pad 105: Net-(A1-Pad105) -> RESET
- A1 pad 107: Net-(A1-Pad107) -> S_CLK
- A1 pad 109: Net-(A1-Pad109) -> S_DATA
- A1 pad 114: (no net) -> Net-(A1-Pad114)
- A1 pad 19: /3V3 -> VDDIO_35
- A1 pad 2: (no net) -> Net-(A1-Pad2)
- A1 pad 20: /3V3 -> VDDIO_35
- A1 pad 61: FLASH -> PMOD1_E
- A1 pad 62: PMOD0_E -> PMOD2_E
- A1 pad 63: SHUTTER -> PMOD0_E
- A1 pad 64: PMOD1_E -> PMOD3_E
- A1 pad 65: SLVS0_P -> EN_S
- A1 pad 66: PMOD2_E -> EN_B
- A1 pad 67: SLVS0_N -> WS2812
- A1 pad 68: PMOD3_E -> EN_A
- A1 pad 70: /1V8 -> VDDIO_34
- A1 pad 71: SLVS1_P -> SHUTTER
- A1 pad 73: SLVS1_N -> CCD_TRIGGER
- A1 pad 75: SLVSC_P -> SLVS0_P
- A1 pad 77: SLVSC_N -> SLVS0_N
- A1 pad 81: /1V8 -> VDDIO_34
- A1 pad 83: SLVS2_P -> SLVS1_P
- A1 pad 85: SLVS2_N -> SLVS1_N
- A1 pad 87: SLVS3_P -> SLVSC_P
- A1 pad 89: SLVS3_N -> SLVSC_N
- A1 pad 93: LED1 -> SLVS2_P
- A1 pad 95: Net-(A1-Pad95) -> SLVS2_N
- A1 pad 97: Net-(A1-Pad97) -> SLVS3_P
- A1 pad 99: Net-(A1-Pad99) -> SLVS3_N
- C1 pad 1: /2V8 -> VDDIO_34
- C1 pad 2: GNDA -> Net-(C1-Pad2)
- C10 pad 1: /1V8 -> Net-(C10-Pad1)
- C11 pad 1: /1V8 -> GNDA
- C11 pad 2: GNDA -> /5V
- C12 pad 1: /1V8 -> /2V8
- C13 pad 1: /1V8 -> /3V3
- C14 pad 1: /2V8 -> /3V3
- C15 pad 1: /1V8 -> /3V3
- C16 pad 1: /1V8 -> /5V
- C17 pad 1: /1V8 -> /5V
- C18 pad 1: /2V8 -> GNDA
- C18 pad 2: GNDA -> /5V
- C19 pad 1: /2V8 -> /1V8
- C2 pad 1: /2V8 -> /3V3
- C2 pad 2: GNDA -> Net-(C1-Pad2)
- C20 pad 1: GNDA -> /3V3
- C20 pad 2: /5V -> GNDA
- C22 pad 1: GNDA -> VDDIO_34
- C22 pad 2: /3V3 -> GNDA
- C23 pad 1: GNDA -> /1V8
- C23 pad 2: /3V3 -> GNDA
- C24 pad 1: GNDA -> /2V8
- C24 pad 2: /1V8 -> GNDA
- C25 pad 1: GNDA -> /2V8
- C25 pad 2: /1V8 -> GNDA
- C26 pad 1: GNDA -> VDDIO_34
- C26 pad 2: /1V8 -> GNDA
- C27 pad 1: /3V3 -> /1V8
- C28 pad 1: /3V3 -> /2V8
- C29 pad 1: /3V3 -> /2V8
- C3 pad 1: /2V8 -> GNDA
- C3 pad 2: GNDA -> /5V
- C4 pad 1: /2V8 -> VDDIO_34
- C5 pad 1: /1V8 -> VDDIO_34
- C6 pad 1: /5V -> VDDIO_34
- C7 pad 1: /1V8 -> GNDA
- C7 pad 2: GNDA -> /5V
- C9 pad 1: /1V8 -> Net-(C8-Pad2)
- C9 pad 2: GNDA -> EN_B
- D1 pad 1: GNDA -> Net-(D1-Pad1)
- D2 pad 1: GNDA -> Net-(D2-Pad1)
- D2 pad 2: Net-(D2-Pad2) -> Net-(D1-Pad1)
- J3 pad 1: Net-(J4-Pad1) (its old number) -> VDDIO_34
- J3 pad 2: Net-(J4-Pad2) (its old number) -> G_ADDR
- J3 pad 3: Net-(J4-Pad3) (its old number) -> GNDA
- R1 pad 1: Net-(A1-Pad105) -> Net-(E1-Pad3)
- R1 pad 2: /1V8 -> EN_A
- R2 pad 1: Net-(A1-Pad107) -> Net-(E1-Pad5)
- R2 pad 2: /1V8 -> EN_B
- R3 pad 1: SLVS0_P -> Net-(E1-Pad3)
- R3 pad 2: SLVS0_N -> VDDIO_35
- R4 pad 1: SLVS1_P -> VDDIO_35
- R4 pad 2: SLVS1_N -> Net-(E1-Pad5)
- R5 pad 1: SLVS2_P -> GNDA
- R5 pad 2: SLVS2_N -> EN_S
- R6 pad 1: SLVS3_P -> Net-(R6-Pad1)
- R6 pad 2: SLVS3_N -> Net-(R6-Pad2)
- R7 pad 1: SLVSC_P -> Net-(R7-Pad1)
- R7 pad 2: SLVSC_N -> Net-(R7-Pad2)
- R8 pad 2: Net-(D1-Pad2) -> Net-(R8-Pad2)
- R9 pad 2: Net-(D2-Pad2) -> Net-(R9-Pad2)
- U1 pad 1: Net-(A1-Pad109) -> VDDIO_35
- U1 pad 2: Net-(A1-Pad107) -> GNDA
- U1 pad 3: FLASH -> WS2812
- U1 pad 4: /1V8 -> Net-(D1-Pad2)
- U1 pad 5: /1V8 -> GNDA
- U1 pad 6: GNDA -> /5V
- U2 pad 1: /5V -> Net-(U2-Pad1)
- U2 pad 2: GNDA -> Net-(U2-Pad2)
- U2 pad 3: /5V -> /3V3
- U2 pad 4: (no net) -> Net-(C1-Pad2)
- U2 pad 5: /2V8 -> Net-(U2-Pad5)
- U3 pad 10: /1V8 -> VDDIO_34
- U3 pad 2: /1V8 -> VDDIO_34
- U4 pad 10: /1V8 -> VDDIO_34
- U4 pad 12: Net-(J4-Pad10) (its old number) -> Net-(J5-Pad10)
- U4 pad 13: Net-(J4-Pad9) (its old number) -> Net-(J5-Pad9)
- U4 pad 14: Net-(J4-Pad8) (its old number) -> Net-(J5-Pad8)
- U4 pad 15: Net-(J4-Pad7) (its old number) -> Net-(J5-Pad7)
- U4 pad 16: Net-(J4-Pad4) (its old number) -> Net-(J5-Pad4)
- U4 pad 17: Net-(J4-Pad3) (its old number) -> Net-(J5-Pad3)
- U4 pad 18: Net-(J4-Pad2) (its old number) -> Net-(J5-Pad2)
- U4 pad 2: /1V8 -> VDDIO_34
- U4 pad 20: Net-(J4-Pad1) (its old number) -> Net-(J5-Pad1)
- U5 pad 10: /1V8 -> VDDIO_34
- U5 pad 12: (no net) -> Net-(U5-Pad12)
- U5 pad 13: (no net) -> Net-(U5-Pad13)
- U5 pad 14: Net-(R9-Pad1) -> Net-(U5-Pad14)
- U5 pad 15: Net-(R8-Pad1) -> Net-(U5-Pad15)
- U5 pad 2: /1V8 -> VDDIO_34
- U5 pad 6: LED1 -> Net-(U5-Pad6)
- U5 pad 7: LED2 -> Net-(U5-Pad7)
- U5 pad 8: (no net) -> Net-(U5-Pad8)
- U5 pad 9: (no net) -> Net-(U5-Pad9)
Routing:
- net GNDA: track 909.9 -> 0.00 mm, vias 52 -> 0
- net /3V3: track 278.6 -> 0.00 mm, vias 6 -> 0
- net /1V8: track 228.6 -> 0.00 mm, vias 3 -> 0
- net /5V: track 178.6 -> 0.00 mm, vias 6 -> 0
- net IO0_N: track 85.8 -> 0.00 mm, vias 1 -> 0
- net IO2_N: track 85.4 -> 0.00 mm, vias 1 -> 0
- net LVDSn0_N: track 81.6 -> 0.00 mm
- net IO1_N: track 80.8 -> 0.00 mm, vias 1 -> 0
- net IO3_N: track 80.7 -> 0.00 mm, vias 1 -> 0
- net SDA_N: track 79.7 -> 0.00 mm, vias 2 -> 0
- net LVDSn4_P: track 79.6 -> 0.00 mm
- net LVDSn0_P: track 77.4 -> 0.00 mm
- net LVDSs0_P: track 76.1 -> 0.00 mm
- net LVDSn1_N: track 75.8 -> 0.00 mm
- net LVDSn5_P: track 75.7 -> 0.00 mm
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- removed copper zone on B.Cu, net GNDA
- removed copper zone on F.Cu, net GNDA
Other:
- board outline removed
- copper layers 2 -> 4
- board text removed: "AXIOM µ"
- board text removed: "v 1.0"
